File: project_gtag.kicad_pcb (KiCad board)
At the start: 2 copper layers, 54 x 30 mm, 14 parts, among them J1 Connector_JTAG, J3 Connector_simple, J4 Connector_compact, SW1 SW_Push

Commit message: Add license, V3.1 and gerbert file
Parts:
- C1: value 10nF -> 100nF
- R4: value 10k -> 1k
- SW1: value SW_Push -> Reset
- TP1: value TestPointGND -> GND
- TP2: value TestPointButton -> VJTAG
Connections:
- net +3V3 renamed /VREF
- net /C2CK renamed /C2CK_TDI
- net /C2D renamed /C2D_TCK
- net /C2Ds renamed /C2Ds_TDO
- C2 pad 1: /C2CKs -> /C2CKs_TMS
- C3 pad 1: /C2CKs -> /C2CKs_TMS
- J1 pad 5: /C2CKs -> /C2CKs_TMS
- J3 pad 4: /C2CKs -> /C2CKs_TMS
- R2 pad 1: /C2CKs -> /C2CKs_TMS
- R4 pad 1: /C2CKs -> /C2CKs_TMS
- SW1 pad 2: /C2CKs -> /C2CKs_TMS
- TP2 pad 1: /C2CKs -> +5V
Routing:
- net /C2CKs: track 62.7 -> 0.00 mm
- net /C2CKs_TMS: track 0.00 -> 57.9 mm
- net +5V: track 12.9 -> 16.9 mm
Other:
- net class Power added: clearance 0.225, trace_width 0.5, via_dia 1.6, via_drill 1
- board text added: "C2CK/TDI"
- board text added: "C2D/TCK"
- board text added: "C2DKs/TMS"
- board text added: "C2Ds/TDO"
- board text added: "G.Guillet 20.05.2020"
- board text added: "GTAG V3.1"
- board text added: "Licensed under CERN OHL v.1.2"
- board text added: "VJTAG"
- board text removed: "C2DKs"
- board text removed: "C2Ds"
- board text removed: "G.Guillet 28.11.2019"
- board text removed: "GTAG V3"
