File: project_gtag.sch (KiCad schematic (older format))
At the start: 14 parts, among them J1 Connector_JTAG, J3 Connector_simple, J4 Connector_compact, SW1 SW_Push

Commit message: Add license, V3.1 and gerbert file
Parts:
- C1: value 10nF -> 100nF
- R4: value 10k -> 1k
- SW1: value SW_Push -> Reset
- TP1: value TestPointGND -> GND
- TP2: value TestPointButton -> VJTAG
Connections:
- net +5V: now also TP2.1
- net +3V3 renamed VREF
- net C2CK renamed C2CK_TDI
- net C2CKs renamed C2CKs_TMS
- net C2CKs_TMS: no longer TP2.1
- net C2D renamed C2D_TCK
- net C2Ds renamed C2Ds_TDO
Other:
- note added: "Compact format"
- note added: "JTAG resistance"
- note added: "Reset button"
- note added: "Silicon-labs, JTAG 2x05 header"
- note added: "Simple format"
- note added: "TestPoints"
- note added: "This documentation describes Open Hardware and is licensed under the\nCERN OHL v. 1.2.\n\nYou may redistribute and modify this documentation under the terms of the\nCERN OHL v.1.2. (http://ohwr.org/cernohl). This documentation is distributed\nWITHOUT ANY EXPRESS OR IMPLIED WARRANTY, INCLUDING OF\nMERCHANTABILITY, SATISFACTORY QUALITY AND FITNESS FOR A\nPARTICULAR PURPOSE. Please see the CERN OHL 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"
- note removed: "Format compact"
- note removed: "Format simple"
- moved on the sheet: C1, C2, C3, D1, J3, J4, R1, R2, R3, SW1, TP1, TP2
